Commit message: First Commit

File: description/robot.urdf.xacro (robot description, xacro)
@@ -1,4 +1,7 @@
 <?xml version="1.0"?>
 <robot xmlns:xacro="http://www.ros.org/wiki/xacro"  name="robot">
-    <xacro:include filename = "robot_core.xacro"/>
+    <xacro:include filename ="robot_core.xacro"/>
+    <xacro:include filename ="gazebo_control.xacro"/>
+    <xacro:include filename ="lidar.xacro"/>
+    <xacro:include filename ="camera.xacro"/>
 </robot>

File: description/robot_core.xacro (robot description, xacro)
@@ -8,4 +8,7 @@
     <material name="orange">
         <color rgba="1 0.3 0.1 1"/>
+    </material>
+    <material name="red">
+        <color rgba="1 0 0 1"/>
     </material>
     <material name="blue">
@@ -44,4 +47,7 @@
         </xacro:inertial_box>
     </link>
+    <gazebo reference="chassis">
+        <material>Gazebo/White</material>
+    </gazebo>
     <!-- Front Left Wheel-->
     <joint name="front_left_wheel_joint" type="continuous">
@@ -68,4 +74,7 @@
         </xacro:inertial_cylinder>
     </link>
+    <gazebo reference="front_left_wheel">
+        <material>Gazebo/Blue</material>
+    </gazebo>
     <!-- Back Left Wheel -->
     <joint name="back_left_wheel_joint" type="continuous">
@@ -92,4 +101,7 @@
         </xacro:inertial_cylinder>
     </link>
+    <gazebo reference="back_left_wheel">
+        <material>Gazebo/Blue</material>
+    </gazebo>
     <!-- Back Right Wheel-->
     <joint name="back_right_wheel_joint" type="continuous">
@@ -116,4 +128,7 @@
         </xacro:inertial_cylinder>
     </link>
+    <gazebo reference="back_right_wheel">
+        <material>Gazebo/Blue</material>
+    </gazebo>
     <!-- Front Right Wheel-->
     <joint name="front_right_wheel_joint" type="continuous">
@@ -140,3 +155,6 @@
         </xacro:inertial_cylinder>
     </link>
+    <gazebo reference="front_right_wheel">
+        <material>Gazebo/Blue</material>
+    </gazebo>
 </robot>
