Commit message: Commit

File: description/gazebo_control.xacro (robot description, xacro)
@@ -2,5 +2,5 @@
 <robot xmlns:xacro="http://www.ros.org/wiki/xacro" >
     <gazebo>
-        <plugin name="wheel_drive_controller" filename="libgazebo_ros_diff_drive.so">
+        <plugin name="diff_drive_controller" filename="libgazebo_ros_diff_drive.so">
             <!-- wheels -->
             <num_wheel_pairs>2</num_wheel_pairs>

File: description/ros2_control.xacro (robot description, xacro)
@@ -2,44 +2,44 @@
 <robot xmlns:xacro="http://www.ros.org/wiki/xacro" >
     <ros2_control name="GazeboSystem" type="system">
-    <hardware>
-        <plugin>gazebo_ros2_control/GazeboSystem</plugin>
-    </hardware>
-    <joint name="front_left_wheel_joint">
-        <command_interface name="velocity">
-            <param name="min">-10</param>
-            <param name="max">10</param>
-        </command_interface>
-        <!-- <state_interface name="position" />
-        <state_interface name="velocity" /> -->
-    </joint>
-    <joint name="back_left_wheel_joint">
-        <command_interface name="velocity">
-            <param name="min">-10</param>
-            <param name="max">10</param>
-        </command_interface>
-        <!-- <state_interface name="position" />
-        <state_interface name="velocity" /> -->
-    </joint>
-    <joint name="front_right_wheel_joint">
-        <command_interface name="velocity">
-            <param name="min">-10</param>
-            <param name="max">10</param>
-        </command_interface>
-        <!-- <state_interface name="velocity" />
-        <state_interface name="position" /> -->
-    </joint>
-    <joint name="back_right_wheel_joint">
-        <command_interface name="velocity">
-            <param name="min">-10</param>
-            <param name="max">10</param>
-        </command_interface>
-        <!-- <state_interface name="velocity" />
-        <state_interface name="position" /> -->
-    </joint>
+        <hardware>
+            <plugin>gazebo_ros2_control/GazeboSystem</plugin>
+        </hardware>
+        <joint name="front_left_wheel_joint">
+            <command_interface name="velocity">
+                <param name="min">-10</param>
+                <param name="max">10</param>
+            </command_interface>
+            <!-- <state_interface name="position" /> -->
+            <!-- <state_interface name="velocity" /> -->
+        </joint>
+        <joint name="back_left_wheel_joint">
+            <command_interface name="velocity">
+                <param name="min">-10</param>
+                <param name="max">10</param>
+            </command_interface>
+            <!-- <state_interface name="position" /> -->
+            <!-- <state_interface name="velocity" /> -->
+        </joint>
+        <joint name="front_right_wheel_joint">
+            <command_interface name="velocity">
+                <param name="min">-10</param>
+                <param name="max">10</param>
+            </command_interface>
+            <!-- <state_interface name="velocity" /> -->
+            <!-- <state_interface name="position" /> -->
+        </joint>
+        <joint name="back_right_wheel_joint">
+            <command_interface name="velocity">
+                <param name="min">-10</param>
+                <param name="max">10</param>
+            </command_interface>
+            <!-- <state_interface name="velocity" /> -->
+            <!-- <state_interface name="position" /> -->
+        </joint>
+    </ros2_control>
     <gazebo>
-        <plugin filename="libgazebo_ros2_control.so" name="gazebo_ros2_control">
-            <parameters>$(find my_bot)/config/my_controllers.yaml</parameters>
+        <plugin name="gazebo_ros2_control" filename="libgazebo_ros2_control.so">
+            <parameters>$(find my_bot)/config/my_controller.yaml</parameters>
         </plugin>
     </gazebo>
-</ros2_control>
 </robot>
